Commit message: 7.11

File: day04_purepursuit/src/pure_pursuit_rviz_demo/urdf/simple_car.urdf (robot description, URDF)
Before this commit: robot simple_car, 5 links, 4 joints
Links:
- removed link left_wheel_link
- removed link right_wheel_link
- added link left_front_wheel_link; visual cylinder length=0.04 radius=0.06
- added link left_rear_wheel_link; visual cylinder length=0.04 radius=0.06
- added link right_front_wheel_link; visual cylinder length=0.04 radius=0.06
- added link right_rear_wheel_link; visual cylinder length=0.04 radius=0.06
- link base_link: geometry visual box size=0.5 0.3 0.1
- link body_link: geometry visual box size=0.35 0.24 0.12
- link front_link: geometry visual box size=0.08 0.22 0.06
Joints:
- removed joint base_to_left_wheel
- removed joint base_to_right_wheel
- added joint base_to_left_front: type fixed, parent base_link, child left_front_wheel_link, origin xyz=0.15 0.17 -0.05 rpy=0 1.5708 0
- added joint base_to_left_rear: type fixed, parent base_link, child left_rear_wheel_link, origin xyz=-0.15 0.17 -0.05 rpy=0 1.5708 0
- added joint base_to_right_front: type fixed, parent base_link, child right_front_wheel_link, origin xyz=0.15 -0.17 -0.05 rpy=0 1.5708 0
- added joint base_to_right_rear: type fixed, parent base_link, child right_rear_wheel_link, origin xyz=-0.15 -0.17 -0.05 rpy=0 1.5708 0
- joint base_to_body: origin xyz=0.0 0.0 0.1 -> xyz=0.0 0.0 0.12
- joint base_to_front: origin xyz=0.2 0.0 0.08 -> xyz=0.29 0.0 0.02
